File: core/esp32 pcb and mounting/pcb files/esp_shield/esp_shield.kicad_pcb (KiCad board)
At the start: 2 copper layers, 162 x 60 mm, 20 parts, among them J1 ESP_01, J10 Relais, J11 BH1750_1, J12 BH1750_2, J13 MH-Z19, J14 Power IN, J15 Power OUT, J16 Conn_02x03_Counter_Clockwise, J17 Conn_01x19, J2 ESP_02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

Commit message: finish wiring + a small change on the pcb + start adding manual
Routing:
- net 1: track 39.1 -> 67.0 mm
Changed lines of the file:
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@@
+	)
+	(segment
+		(start 151.25 124.5)
+		(end 154.323 121.427)
+		(width 0.25)
+		(layer "F.Cu")
+		(net 36)
 	)
 	(segment
 		(start 167 113.5)
 		(end 164.42 110.92)
+		(width 0.25)
+		(layer "F.Cu")
+		(net 36)
+	)
+	(segment
+		(start 134.87 116.75)
+		(end 134.87 120.37)
 		(width 0.25)
 		(layer "F.Cu")
@@
 		(start 156.223 121.427)
 		(end 156.223 113.777)
+		(width 0.25)
+		(layer "F.Cu")
+		(net 36)
+	)
+	(segment
+		(start 154.323 121.427)
+		(end 156.223 121.427)
 		(width 0.25)
 		(layer "F.Cu")
@@
 		(width 0.25)
 		(layer "F.Cu")
+		(net 36)
+	)
+	(segment
+		(start 134.87 120.37)
+		(end 139 124.5)
+		(width 0.25)
+		(layer "F.Cu")
+		(net 36)
+	)
+	(segment
+		(start 139 124.5)
+		(end 151.25 124.5)
+		(width 0.25)
+		(layer "F.Cu")
